File: nwt7.kicad_pcb (KiCad board)
At the start: 2 copper layers, 130 parts, among them IC1 PIC16F876A, IC10 AD8307, IC11 MSA0886, IC12 LM7810CT, IC13 AP1117D50, IC14 AP1117D50, IC15 AP1117D50, IC16 AD8361, IC2 MAX232, IC3 AP1117D50, IC4 AP1117D50, IC5 AP1117D50, IC6 AD9851, IC7 MSA0886, IC8 LM7808CT, IC9 AD8307, P1 IN_LIN, Q1 10 MHz, T1 Coupler

Commit message: ...
Parts:
- moved C13 160.4 mm to (234.4, 94.2), turned to 270 degrees
- moved C22 159.8 mm to (263.3, 74.2), turned to 180 degrees
- moved C21 112.5 mm to (240.7, 84.7)
- moved C31 86.0 mm to (217.2, 97.2), turned to 270 degrees
- moved IC5 11.8 mm to (240.7, 88.3), turned to 180 degrees
- moved R6 3.83 mm to (211.2, 97.2)
- moved R8 2.69 mm to (235.6, 99.9), turned to 180 degrees
Routing:
- net GND: track 27.6 -> 182.5 mm, vias 0 -> 5
- net Net-(C26-Pad1): track 0.00 -> 61.2 mm
- net Net-(C13-Pad2): track 7.03 -> 46.7 mm, vias 0 -> 2
- net Net-(C33-Pad2): track 0.00 -> 12.3 mm
- net Net-(C48-Pad1): track 0.00 -> 12.0 mm
- net Net-(C18-Pad1): track 0.00 -> 12.0 mm
- net Net-(IC6-Pad12): track 3.67 -> 12.6 mm
- net Net-(C24-Pad2): track 0.00 -> 8.29 mm
- net Net-(C29-Pad2): track 0.00 -> 7.30 mm
- net Net-(C34-Pad1): track 0.00 -> 7.28 mm
- net Net-(R31-Pad1): track 0.00 -> 7.28 mm
- net Net-(C4-Pad2): track 0.00 -> 7.20 mm
- net Net-(C51-Pad2): track 0.00 -> 6.69 mm
- net Net-(C51-Pad1): track 0.00 -> 6.60 mm
- net Net-(C49-Pad1): track 0.00 -> 6.43 mm
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
Commit message: ver. 1.0
Parts:
- removed C22, C38, C39: 100nF, Capacitors_SMD:C_1206_HandSoldering
- removed IC14, IC3: AP1117D50, TO_SOT_Packages_SMD:TO-252-2Lead
- C10, C11: footprint Capacitors_SMD:C_1206_HandSoldering -> Capacitors_ThroughHole:C_Disc_D3_P2.5
- C23: footprint Capacitors_SMD:c_elec_5x5.8 -> DDS:CE_Radial_D10_L25_P5
- D3: footprint Diodes_SMD:DO-214AB_Handsoldering -> Discret:D3
- IC11, IC7: footprint TO_SOT_Packages_SMD:TO-50-4_ShortPad-NoHole_Housing -> DDS:Micro-X
- moved C19 137.7 mm to (60.0, 79.3)
- moved IC13 132.8 mm to (46.4, 110.4), turned to 90 degrees
- moved R3 131.7 mm to (43.5, 50.7), turned to 270 degrees
- moved C12 129.1 mm to (43.9, 115.6), turned to 180 degrees
- moved C2 128.1 mm to (110.2, 142.9), turned to 180 degrees
- moved IC11 126.0 mm to (119.1, 113.2), turned to 0 degrees
- moved C37 125.6 mm to (131.8, 91.7)
- moved C8 125.6 mm to (101.6, 35.2), turned to 0 degrees
- moved C17 125.5 mm to (93.6, 114.3)
- moved C26 125.5 mm to (77.0, 130.0)
- moved C28 125.5 mm to (84.1, 116.2)
- moved C34 125.5 mm to (51.6, 121.7)
- moved C36 125.5 mm to (31.2, 130.0)
- moved C42 125.5 mm to (41.4, 124.7)
- moved C49 125.5 mm to (103.8, 114.3)
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Connections:
- R18 pad 2: Net-(IC3-Pad2) -> Net-(C25-Pad1)
- R29 pad 2: Net-(C39-Pad1) -> Net-(C12-Pad2)
Routing:
- net GND: track 182.5 -> 980.2 mm, vias 5 -> 10
- net Net-(C19-Pad2): track 3.67 -> 184.0 mm, vias 0 -> 4
- net Net-(C2-Pad2): track 0.00 -> 175.9 mm
- net Net-(C25-Pad1): track 25.3 -> 156.0 mm, vias 0 -> 4
- net Net-(C37-Pad2): track 0.00 -> 102.0 mm, vias 0 -> 1
- net Net-(C46-Pad2): track 0.00 -> 74.9 mm
- net Net-(C35-Pad1): track 3.07 -> 64.0 mm
- net Net-(IC1-Pad1): track 0.00 -> 31.1 mm
- net Net-(D1-Pad1): track 0.00 -> 30.8 mm
- net Net-(IC1-Pad28): track 0.00 -> 20.7 mm
- net Net-(IC1-Pad27): track 0.00 -> 20.3 mm
- net Net-(C12-Pad2): track 3.37 -> 18.6 mm
- net Net-(R34-Pad1): track 0.00 -> 14.4 mm
- net Net-(C40-Pad1): track 0.00 -> 13.2 mm
- net Net-(C44-Pad1): track 0.00 -> 12.3 mm
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- added copper zone on B.Cu, net GND
- added copper zone on F.Cu, net GND

Commit message: edge cuts
Other:
- board outline added: 120.7 x 117.3 mm
- rule pad_to_mask_clearance: 0.2 -> 0.1
Changed lines of the file:
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@@
     (links 255)
     (no_connects 0)
-    (area 0 0 0 0)
+    (area 26.434 21.949999 147.152 166.167481)
     (thickness 1.6)
-    (drawings 0)
+    (drawings 4)
     (tracks 802)
     (zones 0)
@@
     (pad_size 3.6 1.8)
     (pad_drill 1)
-    (pad_to_mask_clearance 0.2)
+    (pad_to_mask_clearance 0.1)
     (aux_axis_origin 0 0)
     (grid_origin 220.047 92.004)
     (visible_elements FFFFFF7F)
     (pcbplotparams
-      (layerselection 0x00030_80000001)
-      (usegerberextensions false)
-      (excludeedgelayer true)
+      (layerselection 0x010f0_80000001)
+      (usegerberextensions true)
+      (excludeedgelayer false)
       (linewidth 0.100000)
       (plotframeref false)
@@
       (outputformat 1)
       (mirror false)
-      (drillshape 1)
+      (drillshape 0)
       (scaleselection 1)
       (outputdirectory ""))
@@
     )
   )
+  (gr_line (start 147.149 30.028) (end 26.499 30.028) (angle 90) (layer Edge.Cuts) (width 0.15))
+  (gr_line (start 147.149 147.376) (end 147.149 30.028) (angle 90) (layer Edge.Cuts) (width 0.15))
+  (gr_line (start 26.499 147.376) (end 147.149 147.376) (angle 90) (layer Edge.Cuts) (width 0.15))
+  (gr_line (start 26.499 30.028) (end 26.499 147.376) (angle 90) (layer Edge.Cuts) (width 0.15))
   (segment (start 99.092 56.007) (end 97.822 56.007) (width 0.4) (layer F.Cu) (net 1))
   (segment (start 97.822 56.007) (end 94.901 53.086) (width 0.4) (layer F.Cu) (net 1))

Commit message: ...
Parts:
- removed P1: IN_LIN, Sockets_BNC:BNC_Socket_TYCO-AMP_LargePads
- added ST4: IN_LIN, DDS:BNC_Socket_Base, F.Cu at (38.9, 121.5)
- C1, C2, C6, C7, C8, C9: value 1uF -> 1u
- C12, C13, C15, C19, C21, C24, C25, C26, C27, C28, C29, C3, C31, C33, C36, C4, C40, C41, C42, C43, C44, C45, C47, C5, C51, C52, C53, C54: value 100nF -> 100n
- C14: value 10uF -> 10u
- C16, C17, C18, C48, C49, C50: value 60pF -> 60p
- C34, C35, C37, C46: value 1nF -> 1n
- L1, L2, L4, L5: value 180nH -> 180n
- L3, L6: value 10uH -> 10u
- ST1, ST2, ST6: footprint Sockets_BNC:BNC_Socket_TYCO-AMP_LargePads -> DDS:BNC_Socket_Base
- ST3: footprint Connect:DB9MC -> DDS:DB9_Base
- moved C13 22.6 mm to (95.4, 65.2)
- moved C16 22.6 mm to (79.5, 85.2)
- moved C18 22.6 mm to (79.5, 108.1)
- moved C2 22.6 mm to (96.1, 125.2)
- moved C27 22.6 mm to (70.6, 43.8)
- moved L2 22.6 mm to (77.6, 102.4)
- moved L3 22.6 mm to (60.8, 99.9)
- moved L4 22.6 mm to (91.6, 102.4)
- moved R15 22.6 mm to (60.8, 106.6)
- moved R16 22.6 mm to (106.2, 33.8)
- moved R2 22.6 mm to (106.2, 39.4)
- moved R33 22.6 mm to (127.4, 77.2)
- moved R34 22.6 mm to (119.5, 108.6)
- moved R35 22.6 mm to (119.5, 96.1)
- moved R39 22.6 mm to (99.2, 108.1)
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Other:
- board size 120.7 x 117.3 mm -> 120.6 x 117.3 mm

Commit message: fixed pcb
Other:
- board text added: "NWT 7 PCB design by Paweł SQ5KVP"

Commit message: polishing pcb
Routing:
- net GND: track 980.2 -> 110.2 mm, vias 10 -> 8

Commit message: ...
Parts:
- IC12: value LM7810CT -> 78L10; footprint TO_SOT_Packages_THT:TO-220_Neutral123_Horizontal_LargePads -> TO_SOT_Packages_THT:TO-92_Rugged
- IC8: value LM7808CT -> 7808
- R15, R42: value 180 -> 68
- T1: footprint Choke_Toroid_ThroughHole:Transformer_Toroid_horizontal_Diameter10-5mm_Amidon-T37 -> DDS:Transformer_Amidon-T37
- moved C2 5.24 mm to (98.0, 120.3), turned to 270 degrees
- moved IC12 2.34 mm to (94.1, 122.1)
Routing:
- net Net-(C19-Pad2): track 184.0 -> 182.4 mm
- net Net-(C2-Pad2): track 175.9 -> 176.9 mm
Other:
- board text added: "NWT 7 PCB design by Paweł A. Ryszawa SQ5KVP"
- board text removed: "NWT 7 PCB design by Paweł SQ5KVP"

Commit message: fix
Parts:
- moved IC12 4.95 mm to (94.1, 117.2), turned to 270 degrees
- moved C2 1.78 mm to (99.8, 120.2)
Connections:
- IC12 pad 1: Net-(C2-Pad2) -> Net-(C26-Pad1)
- IC12 pad 3: Net-(C26-Pad1) -> Net-(C2-Pad2)
Routing:
- net Net-(C2-Pad2): track 176.9 -> 178.7 mm
