File: nwt7.kicad_pcb (KiCad board)
At the start: 2 copper layers, 120.6 x 117.3 mm, 125 parts, among them IC1 PIC16F876A, IC10 AD8307, IC11 MSA0886, IC12 78L10, IC13 AP1117D50, IC15 AP1117D50, IC16 AD8361, IC2 MAX232, IC4 AP1117D50, IC5 AP1117D50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

Commit message: narrowed PCB
Parts:
- moved IC8 2.67 mm to (22.6, 44.0)
- moved C36 1.40 mm to (18.5, 112.4)
- moved C42 1.40 mm to (28.7, 107.1)
- moved C46 1.40 mm to (26.7, 102.5)
- moved R29 1.40 mm to (22.4, 99.6)
- moved ST1 1.40 mm to (22.6, 121.5)
- moved C40 1.40 mm to (18.8, 102.5)
- moved IC9 1.40 mm to (22.1, 107.1)
- moved R30 1.40 mm to (25.4, 112.4)
- moved T1 0.76 mm to (126.1, 100.7)
Routing:
- net Net-(C2-Pad2): track 178.7 -> 173.7 mm
- net Net-(C19-Pad2): track 182.4 -> 177.4 mm
- net Net-(C40-Pad1): track 13.2 -> 16.2 mm
- net Net-(C46-Pad2): track 74.9 -> 77.5 mm
- net Net-(C33-Pad2): track 12.3 -> 14.8 mm
- net Net-(C12-Pad2): track 18.6 -> 17.2 mm
- net Net-(C36-Pad2): track 4.82 -> 5.98 mm
- net Net-(R34-Pad1): track 14.4 -> 13.9 mm
Other:
- board size 120.6 x 117.3 mm -> 118.4 x 117.3 mm

Commit message: adjusting
Parts:
- added REF**: Hole3, DDS:Hole3, F.Cu at (28.1, 44.1)
- added REF**: Hole3, DDS:Hole3, F.Cu at (115.1, 44.1)
- added REF**: Hole3, DDS:Hole3, F.Cu at (72.0, 122.2)
- moved ST3 1.55 mm to (110.8, 20.5)
- moved C15 1.55 mm to (75.9, 80.3)
- moved C16 1.55 mm to (78.0, 85.0)
- moved C17 1.55 mm to (78.0, 96.4)
- moved C18 1.55 mm to (78.0, 107.8)
- moved C19 1.55 mm to (44.4, 61.4)
- moved C28 1.55 mm to (68.5, 98.3)
- moved C3 1.55 mm to (90.2, 80.3)
- moved C31 1.55 mm to (76.6, 67.8)
- moved C32 1.55 mm to (90.3, 58.5)
- moved C34 1.55 mm to (35.9, 103.8)
- moved C35 1.55 mm to (38.5, 97.7)
- moved C40 1.55 mm to (17.3, 102.2)
- moved C42 1.55 mm to (27.2, 106.8)
- moved C43 1.55 mm to (128.7, 80.9)
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Other:
- board size 118.4 x 117.3 mm -> 119.1 x 117.3 mm
